File: Rev A/BatteryChargingModule_Mainboard.kicad_sch (KiCad schematic)
At the start: 0 parts

Commit message: yes
Parts:
- added H10, H11, H12, H17, H9: M3x11 Standoff, Mounting_Wuerth:Mounting_Wuerth_WA-SMSI-M3_H11mm_9774110360, symbol Mechanical:MountingHole_Pad
- added J6: 2x7 P2.54mm, Connector_PinSocket_2.54mm:PinSocket_2x07_P2.54mm_Vertical, symbol Connector_Generic:Conn_02x07_Odd_Even
Connections:
- new net BAT+: H11.1
- new net BAT-: H12.1
- new net BOOST +24V: H17.1
- new net EA2+: J6.6 (Pin_6)
- new net GND: H10.1
- new net IRef: J6.3 (Pin_3)
- new net SOLAR+: H9.1
- new net SolarSense: J6.9 (Pin_9)
- new net VRef: J6.1 (Pin_1)
Other:
- note added: "Header Connection (MCU Input) and Test Points"
