File: Rev A/MCUModule.kicad_sch (KiCad schematic)
At the start: 0 parts

Commit message: yes
Parts:
- added H5, H6, H7, H8: M3x11 Standoff, Mounting_Wuerth:Mounting_Wuerth_WA-SMSI-M3_H11mm_9774110360, symbol Mechanical:MountingHole_Pad
- added J2, J3: 2x7 P2.54mm, Connector_PinSocket_2.54mm:PinSocket_2x07_P2.54mm_Vertical, symbol Connector_Generic:Conn_02x07_Odd_Even
- added SYM3: SYM_Hot_Small, Modules_SurgicalLighting:MCUModule, symbol Graphic:SYM_Hot_Small
Connections:
- new net 12V_Battery: H7.1
- new net 12V_Wall: H8.1
- new net BatChgEna1: J2.7 (Pin_7)
- new net BatChgEna2: J2.9 (Pin_9)
- new net BoostEna1: J2.3 (Pin_3)
- new net BoostEna2: J2.5 (Pin_5)
- new net BoostVoltage_0.1x: J3.7 (Pin_7), J3.8 (Pin_8)
- new net DisableBackupPico: J2.2 (Pin_2)
- new net GND: H5.1, J2.14 (Pin_14)
- new net IRef_Buck: J2.11 (Pin_11)
- new net IsenBatChg: J3.1 (Pin_1), J3.2 (Pin_2)
- new net LightISense1: J3.5 (Pin_5), J3.6 (Pin_6)
- new net LightISense2: J3.3 (Pin_3), J3.4 (Pin_4)
- new net ModuleENA: J2.1 (Pin_1)
- new net PWM_Lights1: J2.8 (Pin_8)
- new net PWM_Lights2: J2.10 (Pin_10)
- new net PowerModuleEna1: J2.4 (Pin_4)
- new net PowerModuleEna2: J2.6 (Pin_6)
- new net RelaySelectHighPreference: J2.12 (Pin_12)
- new net SOLAR: H6.1
- new net SolarSense: J3.10 (Pin_10), J3.9 (Pin_9)
- new net VRef_Buck: J2.13 (Pin_13)
Other:
- note added: "Mounting Holes for Power Connections"
