File: Rev A/Mainboard.kicad_pcb (KiCad board)
At the start: 2 copper layers, 0 parts

Commit message: Added power Module, started layout
Parts:
- added D1: PESD3V3L1BA,115, Diode_SMD:D_SOD-323F, F.Cu at (81.0, 83.0)
- added D2: PESD3V3L1BA,115, Diode_SMD:D_SOD-323F, F.Cu at (81.0, 86.0)
- added D3: PESD3V3L1BA,115, Diode_SMD:D_SOD-323F, F.Cu at (81.0, 88.9)
- added D4: PESD3V3L1BA,115, Diode_SMD:D_SOD-323F, F.Cu at (81.0, 91.8)
- added D5: PESD3V3L1BA,115, Diode_SMD:D_SOD-323F, F.Cu at (81.0, 94.8)
- added H1: M3x11 Standoff, Mounting_Wuerth:Mounting_Wuerth_WA-SMSI-M3_H11mm_9774110360, F.Cu at (77.0, 133.0)
- added H2: M3x11 Standoff, Mounting_Wuerth:Mounting_Wuerth_WA-SMSI-M3_H11mm_9774110360, F.Cu at (167.0, 133.0)
- added H3: M3x11 Standoff, Mounting_Wuerth:Mounting_Wuerth_WA-SMSI-M3_H11mm_9774110360, F.Cu at (77.0, 43.0)
- added H4: M3x11 Standoff, Mounting_Wuerth:Mounting_Wuerth_WA-SMSI-M3_H11mm_9774110360, F.Cu at (167.0, 43.0)
- added J1: 1x7 Socket P2.54mm, Connector_PinHeader_2.54mm:PinHeader_1x07_P2.54mm_Vertical, F.Cu at (77.0, 80.4)
- added SYM1: Logo_Open_Hardware_Large, Symbol:OSHW-Logo_38.1x40mm_SilkScreen, F.Cu at (22.0, 188.0)
Other:
- board outline added: 279 x 239 mm
- board text added: "Mainboard"
- board text added: "Power Module"

Commit message: yes
Parts:
- removed D1, D2, D3, D4, D5: PESD3V3L1BA,115, Diode_SMD:D_SOD-323F
- added H10: M3x11 Standoff, Mounting_Wuerth:Mounting_Wuerth_WA-SMSI-M3_H11mm_9774110360, F.Cu at (-234.0, 185.0)
- added H11: M3x11 Standoff, Mounting_Wuerth:Mounting_Wuerth_WA-SMSI-M3_H11mm_9774110360, F.Cu at (-234.0, 165.9)
- added H12: M3x11 Standoff, Mounting_Wuerth:Mounting_Wuerth_WA-SMSI-M3_H11mm_9774110360, F.Cu at (-109.6, 165.9)
- added H13: M3x11 Standoff, Mounting_Wuerth:Mounting_Wuerth_WA-SMSI-M3_H11mm_9774110360, F.Cu at (-106.8, 57.1)
- added H14: M3x11 Standoff, Mounting_Wuerth:Mounting_Wuerth_WA-SMSI-M3_H11mm_9774110360, F.Cu at (-236.8, 57.1)
- added H15: M3x11 Standoff, Mounting_Wuerth:Mounting_Wuerth_WA-SMSI-M3_H11mm_9774110360, F.Cu at (-236.8, 137.2)
- added H16: M3x11 Standoff, Mounting_Wuerth:Mounting_Wuerth_WA-SMSI-M3_H11mm_9774110360, F.Cu at (-106.8, 137.2)
- added H17: M3x11 Standoff, Mounting_Wuerth:Mounting_Wuerth_WA-SMSI-M3_H11mm_9774110360, F.Cu at (-104.5, 207.4)
- added H5: M3x11 Standoff, Mounting_Wuerth:Mounting_Wuerth_WA-SMSI-M3_H11mm_9774110360, F.Cu at (-59.3, 246.5)
- added H6: M3x11 Standoff, Mounting_Wuerth:Mounting_Wuerth_WA-SMSI-M3_H11mm_9774110360, F.Cu at (-59.3, 166.5)
- added H7: M3x11 Standoff, Mounting_Wuerth:Mounting_Wuerth_WA-SMSI-M3_H11mm_9774110360, F.Cu at (20.7, 166.5)
- added H8: M3x11 Standoff, Mounting_Wuerth:Mounting_Wuerth_WA-SMSI-M3_H11mm_9774110360, F.Cu at (15.7, 246.5)
- added H9: M3x11 Standoff, Mounting_Wuerth:Mounting_Wuerth_WA-SMSI-M3_H11mm_9774110360, F.Cu at (-104.5, 184.5)
- added J2: 2x7 P2.54mm, Connector_PinSocket_2.54mm:PinSocket_2x07_P2.54mm_Vertical, F.Cu at (-58.0, 198.9)
- added J3: 2x7 P2.54mm, Connector_PinSocket_2.54mm:PinSocket_2x07_P2.54mm_Vertical, F.Cu at (21.9, 198.9)
- added J4: NC6-P108-02, Connectors_SurgicalLighting:NC6-P108-02, F.Cu at (-253.1, 90.4)
- added J5: 2x7 P2.54mm, Connector_PinSocket_2.54mm:PinSocket_2x07_P2.54mm_Vertical, F.Cu at (-171.9, 135.9)
- added J6: 2x7 P2.54mm, Connector_PinSocket_2.54mm:PinSocket_2x07_P2.54mm_Vertical, F.Cu at (-194.7, 167.2)
- added J7: NC6-P108-02, Connectors_SurgicalLighting:NC6-P108-02, F.Cu at (-253.1, 229.4)
- added J8: NC6-P108-02, Connectors_SurgicalLighting:NC6-P108-02, F.Cu at (-253.1, 166.3)
- added SYM2: SYM_Hot_Small, Modules_SurgicalLighting:PowerModule, F.Cu at (-16.9, 92.3)
- added SYM3: SYM_Hot_Small, Modules_SurgicalLighting:MCUModule, F.Cu at (-64.3, 251.5)
- added U1: TL494, Package_DIP:DIP-16_W7.62mm_Socket, F.Cu at (-177.7, 60.7)
- added kibuzzard-662287CC: G***, kibuzzard-662287CC, F.Cu at (-52.7, 115.0)
- added kibuzzard-662C5ACC: G***, kibuzzard-662C5ACC, F.Cu at (-247.2, 18.9)
- J1: value 1x7 Socket P2.54mm -> 2x7 P2.54mm; footprint Connector_PinHeader_2.54mm:PinHeader_1x07_P2.54mm_Vertical -> Connector_PinSocket_2.54mm:PinSocket_2x07_P2.54mm_Vertical
- SYM1: value Logo_Open_Hardware_Large -> SYM_Hot_Small; footprint Symbol:OSHW-Logo_38.1x40mm_SilkScreen -> Modules_SurgicalLighting:BoostModule
- moved SYM1 267.7 mm to (-241.7, 142.3)
- moved H1 139.0 mm to (-61.9, 137.3)
- moved H2 139.0 mm to (28.1, 137.3)
- moved H3 139.0 mm to (-61.9, 47.3)
- moved H4 139.0 mm to (28.1, 47.3)
- moved J1 138.2 mm to (-61.1, 84.7)
Connections:
- H3 pad 1: /Power Module/12V_LowPreference -> BAT+
- H4 pad 1: /Power Module/12V_HighPreference -> +12V
- J1 pad 2: /Power Module/RelaySelectHighPreference -> unconnected-(J1-Pin_1-Pad1)
- J1 pad 3: /Power Module/PWM_Lights1 -> /Relay
- J1 pad 4: /Power Module/PWM_Lights2 -> /Relay
- J1 pad 5: /Power Module/CurrentSenseCh1 -> /PWM1
- J1 pad 6: /Power Module/CurrentSenseCh2 -> /PWM1
- J1 pad 7: GND -> /PWM2
Routing:
- net +12V: track 0.00 -> 509.1 mm
- net BAT+: track 0.00 -> 415.7 mm
- net SOLAR+: track 0.00 -> 355.6 mm, vias 0 -> 2
- net /ISenBatChg: track 0.00 -> 346.2 mm
- net /SolarSense: track 0.00 -> 337.9 mm, vias 0 -> 1
- net /BSTEna: track 0.00 -> 263.2 mm
- net IRef: track 0.00 -> 262.2 mm, vias 0 -> 2
- net VRef: track 0.00 -> 259.1 mm, vias 0 -> 2
- net +24V: track 0.00 -> 167.6 mm
- net BAT-: track 0.00 -> 160.7 mm
- net /ISen2: track 0.00 -> 155.8 mm
- net /ISen1: track 0.00 -> 147.6 mm
- net /Relay: track 0.00 -> 137.8 mm
- net /PWM1: track 0.00 -> 128.1 mm
- net /PWM2: track 0.00 -> 126.0 mm, vias 0 -> 1
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- added copper zone on F.Cu, net +12V
- added copper zone on F.Cu, net +24V
- added copper zone on F.Cu, net BAT+
- added copper zone on F.Cu, net BAT-
- added copper zone on B.Cu, net GND
- added copper zone on F.Cu, net GND
- added copper zone on F.Cu, net SOLAR+
Other:
- board size 279 x 239 mm -> 320 x 254 mm
- board text added: "+BAT"
- board text added: "+SOLAR"
- board text added: "-BAT"
- board text added: "Battery Charging Module"
- board text added: "Boost Converter Module"
- board text added: "GND"
- board text added: "I HATE THIS FUCKING PCB"
- board text added: "MCU Module"
- board text added: "Spare TL494 for replacement Under Boost PCB"
- board text added: "Wall 12V"
- board text added: "i just wanna graduatteee"
- board text added: "it's joever"
- board text added: "what the fuck am I doing"
- board text removed: "Mainboard"
